Commit message: Working commits.

File: examples/RimlessTorso/SkinnyTorsoBalance.urdf (robot description, URDF)
Before this commit: robot TorsoBalance, 9 links, 8 joints
Links:
- link center: geometry visual cylinder length=.1 radius=0.02; visual sphere radius=.06
- link leg1: geometry visual cylinder length=1 radius=0.02
- link leg2: geometry visual cylinder length=1 radius=0.02
- link toe1: geometry collision sphere radius=0; visual sphere radius=0.015
- link toe2: geometry collision sphere radius=0; visual sphere radius=0.015
- link torso: geometry visual cylinder length=.75 radius=0.02
